Commit message: [update] add zm description

File: junbot/junbot_mecanum_description/urdf/turtlebot3_mecanum.urdf.xacro (robot description, xacro)
@@ -1,5 +1,6 @@
 <?xml version="1.0" ?>
 <robot name="turtlebot3_mecanum" xmlns:xacro="http://ros.org/wiki/xacro">
-  <xacro:include filename="$(find turtlebot3_description)/urdf/common_properties.xacro"/>
+  <xacro:include filename="$(find junbot_mecanum_description)/urdf/common_properties.xacro"/>
+  <xacro:include filename="$(find junbot_mecanum_description)/urdf/turtlebot3_mecanum.gazebo.xacro"/>
   <link name="base_footprint"/>
 	<joint name="base_joint" type="fixed">
@@ -12,5 +13,5 @@
 			<origin xyz="0.0355 0 0" rpy="0 0 0" />
 			<geometry>
-				<mesh filename="package://turtlebot3_description/meshes/bases/base_link.STL" />
+				<mesh filename="package://junbot_mecanum_description/meshes/bases/base_link.STL" />
 			</geometry>
 			<material name="light_black">
@@ -21,5 +22,5 @@
 			<origin xyz="0 0 0" rpy="0 0 0" />
 			<geometry>
-				<mesh filename="package://turtlebot3_description/meshes/bases/base_link.STL" />
+				<mesh filename="package://junbot_mecanum_description/meshes/bases/base_link.STL" />
 			</geometry>
 		</collision>
@@ -46,5 +47,5 @@
 			<origin xyz="0 0 -0.009" rpy="0 1.57 0"/>
      			<geometry>
-				<mesh filename="package://turtlebot3_description/meshes/wheels/wheel_right_rear.STL" />
+				<mesh filename="package://junbot_mecanum_description/meshes/wheels/wheel_right_rear.STL" />
 			</geometry>
    			<material name="dark">
@@ -55,5 +56,5 @@
 			<origin xyz="0 0 0" rpy="0 0 0" />
 			<geometry>
-				<mesh filename="package://turtlebot3_description/meshes/wheels/wheel_right_rear.STL" />
+				<mesh filename="package://junbot_mecanum_description/meshes/wheels/wheel_right_rear.STL" />
 			</geometry>
 		</collision>
@@ -80,5 +81,5 @@
 			<origin xyz="0 0 0.009" rpy="0 1.57 0 "/>
      			<geometry>
-				<mesh filename="package://turtlebot3_description/meshes/wheels/wheel_left_rear.STL" />
+				<mesh filename="package://junbot_mecanum_description/meshes/wheels/wheel_left_rear.STL" />
 			</geometry>
    			<material name="Rubber">
@@ -89,5 +90,5 @@
 			<origin xyz="0 0 0" rpy="0 0 0" />
 			<geometry>
-				<mesh filename="package://turtlebot3_description/meshes/wheels/wheel_left_rear.STL" />
+				<mesh filename="package://junbot_mecanum_description/meshes/wheels/wheel_left_rear.STL" />
 			</geometry>
 		</collision>
@@ -114,5 +115,5 @@
 			<origin xyz="0 0 -0.009" rpy="0 1.57 0"/>
      			<geometry>
-				<mesh filename="package://turtlebot3_description/meshes/wheels/wheel_right_front.STL" />
+				<mesh filename="package://junbot_mecanum_description/meshes/wheels/wheel_right_front.STL" />
 			</geometry>
    			<material name="Rubber">
@@ -123,5 +124,5 @@
 			<origin xyz="0 0 0" rpy="0 0 0" />
 			<geometry>
-				<mesh filename="package://turtlebot3_description/meshes/wheels/wheel_right_front.STL" />
+				<mesh filename="package://junbot_mecanum_description/meshes/wheels/wheel_right_front.STL" />
 			</geometry>
 		</collision>
@@ -148,5 +149,5 @@
 			<origin xyz="0 0 0.009" rpy="0 1.57 0"/>
      			<geometry>
-				<mesh filename="package://turtlebot3_description/meshes/wheels/wheel_left_front.STL" />
+				<mesh filename="package://junbot_mecanum_description/meshes/wheels/wheel_left_front.STL" />
 			</geometry>
    			<material name="Rubber">
@@ -157,5 +158,5 @@
 			<origin xyz="0 0 0" rpy="0 0 0" />
 			<geometry>
-				<mesh filename="package://turtlebot3_description/meshes/wheels/wheel_left_front.STL" />
+				<mesh filename="package://junbot_mecanum_description/meshes/wheels/wheel_left_front.STL" />
 			</geometry>
 		</collision>
@@ -190,5 +191,5 @@
       <origin xyz="0 0 0.03" rpy="0 0 0"/>
       <geometry>
-        <mesh filename="package://turtlebot3_description/meshes/bases/lds.STL" scale="0.001 0.001 0.001"/>
+        <mesh filename="package://junbot_mecanum_description/meshes/bases/lds.STL" scale="0.001 0.001 0.001"/>
       </geometry>
       <material name="dark"/>
