Commit message: [update] fix urdf

File: junbot/junbot_description/urdf/junbot_mecanum.urdf.xacro (robot description, xacro)
@@ -87,5 +87,5 @@
     <parent link="base_link"/>
     <child link="sick_lidar0"/>
-    <origin xyz="0.33 0.175 0.195722" rpy="0 0 0.7854"/>
+    <origin xyz="0.2 0 0.195722" rpy="0 0 0"/>
   </joint>
   <link name="sick_lidar0">
@@ -112,5 +112,5 @@
   </link>
   <!-- sick LiDAR 1 -->
-  <joint name="sick_lidar1_joint" type="fixed">
+  <!-- <joint name="sick_lidar1_joint" type="fixed">
     <parent link="base_link"/>
     <child link="sick_lidar1"/>
@@ -138,10 +138,10 @@
 	             izz="0.0001"/>
       </inertial>
-  </link>
+  </link> -->
   <!-- kinect V2 -->
   <joint name="kinect_v2_joint " type="fixed">
     <parent link="base_link"/>
     <child link="kinect_v2"/>
-    <origin xyz="0.297 -0.05 0.122015" rpy="0 0 0"/>
+    <origin xyz="0.33 0 0.122015" rpy="0 0 0"/>
     <axis xyz="0 0 1"/>
   </joint>

Commit message: [Fixed] remove sonar map layer

File: junbot/junbot_description/urdf/junbot_mecanum.urdf.xacro (robot description, xacro)
@@ -10,5 +10,5 @@
   <xacro:property name="wheel_right_W" value="-0.3" /> <!-- wheel right W -->
   <!-- ultrasound position on robot-->
-  <xacro:property name="ul_left_front_x" value="0.4"/>
+  <!-- <xacro:property name="ul_left_front_x" value="0.4"/>
   <xacro:property name="ul_left_front_y" value="0.15" />
   <xacro:property name="ul_right_front_x" value="0.4" />
@@ -20,5 +20,5 @@
   <xacro:property name="ul_hight" value="0.03" />
   <xacro:property name="ul_front_rotation" value="0" />
-  <xacro:property name="ul_rear_rotation" value="3.141592654" />
+  <xacro:property name="ul_rear_rotation" value="3.141592654" /> -->
   <!-- roller position -->
   <xacro:property name="roller_1_y" value="0"/>
@@ -49,5 +49,5 @@
   <xacro:include filename="$(find junbot_description)/urdf/junbot_wheel_RR.urdf.xacro"/>
   <!-- Import Ultrasound -->
-  <xacro:include filename="$(find junbot_description)/urdf/junbot_ultrasound.urdf.xacro"/>
+  <!-- <xacro:include filename="$(find junbot_description)/urdf/junbot_ultrasound.urdf.xacro"/> -->
   <!-- Import Plugin -->
   <xacro:include filename="$(find junbot_description)/urdf/junbot_plugin.gazebo"/>
@@ -400,5 +400,5 @@
   <xacro:roller_trans_v0 prefix="roller_4_8"/>
   <xacro:roller_trans_v0 prefix="roller_4_9"/>
-  <!-- ultrasound -->
+  <!-- ultrasound
   <xacro:zm_ultrasound prefix="1" parent="base_link" origin_x="${ul_left_front_x}" origin_y="${ul_left_front_y}"
                                                      origin_z="${ul_hight}" rotation_z="${ul_front_rotation}">
@@ -412,4 +412,4 @@
   <xacro:zm_ultrasound prefix="4" parent="base_link" origin_x="${ul_right_rear_x}" origin_y="${ul_right_rear_y}"
                                                      origin_z="${ul_hight}" rotation_z="${ul_rear_rotation}">
-  </xacro:zm_ultrasound>
+  </xacro:zm_ultrasound> -->
 </robot>
