Commit message: [fixed] change name to junbot

File: junbot/junbot_description/urdf/junbot_mecanum.urdf.xacro (robot description, xacro)
@@ -197,128 +197,128 @@
     </inertial>
   </link>
-  <!--zm robot LR wheel-->
-  <xacro:zm_wheel_v1 prefix="1" parent="base_link" origin_x="${wheel_after_L}" origin_y="${wheel_left_W}" rotation_x="${wheel_rotationx}">
-  </xacro:zm_wheel_v1>
-  <!--zm robot LR rollor-->
-  <xacro:zm_roller_v0 prefix="roller_1_1" parent="wheel_1" origin_x="${roller_1_y}" origin_y="${roller_1_x}"
+  <!--junbot robot LR wheel-->
+  <xacro:junbot_wheel_v1 prefix="1" parent="base_link" origin_x="${wheel_after_L}" origin_y="${wheel_left_W}" rotation_x="${wheel_rotationx}">
+  </xacro:junbot_wheel_v1>
+  <!--junbot robot LR rollor-->
+  <xacro:junbot_roller_v0 prefix="roller_1_1" parent="wheel_1" origin_x="${roller_1_y}" origin_y="${roller_1_x}"
                                                            rotation_x="0.7854" rotation_z="1.5708">
-  </xacro:zm_roller_v0>
-  <xacro:zm_roller_v0 prefix="roller_1_2" parent="wheel_1" origin_x="${roller_2_y}" origin_y="${roller_2_x}"
+  </xacro:junbot_roller_v0>
+  <xacro:junbot_roller_v0 prefix="roller_1_2" parent="wheel_1" origin_x="${roller_2_y}" origin_y="${roller_2_x}"
                                                            rotation_x="0.7854" rotation_z="0.8727">
-  </xacro:zm_roller_v0>
-  <xacro:zm_roller_v0 prefix="roller_1_3" parent="wheel_1" origin_x="${roller_3_y}" origin_y="${roller_3_x}"
+  </xacro:junbot_roller_v0>
+  <xacro:junbot_roller_v0 prefix="roller_1_3" parent="wheel_1" origin_x="${roller_3_y}" origin_y="${roller_3_x}"
                                                            rotation_x="0.7854" rotation_z="0.1746">
-  </xacro:zm_roller_v0>
-  <xacro:zm_roller_v0 prefix="roller_1_4" parent="wheel_1" origin_x="${roller_4_y}" origin_y="${roller_4_x}"
+  </xacro:junbot_roller_v0>
+  <xacro:junbot_roller_v0 prefix="roller_1_4" parent="wheel_1" origin_x="${roller_4_y}" origin_y="${roller_4_x}"
                                                            rotation_x="0.7854" rotation_z="-0.5235">
-  </xacro:zm_roller_v0>
-  <xacro:zm_roller_v0 prefix="roller_1_5" parent="wheel_1" origin_x="${roller_5_y}" origin_y="${roller_5_x}"
+  </xacro:junbot_roller_v0>
+  <xacro:junbot_roller_v0 prefix="roller_1_5" parent="wheel_1" origin_x="${roller_5_y}" origin_y="${roller_5_x}"
                                                            rotation_x="0.7854" rotation_z="-1.2216">
-  </xacro:zm_roller_v0>
-  <xacro:zm_roller_v0 prefix="roller_1_6" parent="wheel_1" origin_x="${roller_6_y}" origin_y="${roller_6_x}"
+  </xacro:junbot_roller_v0>
+  <xacro:junbot_roller_v0 prefix="roller_1_6" parent="wheel_1" origin_x="${roller_6_y}" origin_y="${roller_6_x}"
                                                            rotation_x="0.7854" rotation_z="4.3632">
-  </xacro:zm_roller_v0>
-  <xacro:zm_roller_v0 prefix="roller_1_7" parent="wheel_1" origin_x="${roller_7_y}" origin_y="${roller_7_x}"
+  </xacro:junbot_roller_v0>
+  <xacro:junbot_roller_v0 prefix="roller_1_7" parent="wheel_1" origin_x="${roller_7_y}" origin_y="${roller_7_x}"
                                                            rotation_x="0.7854" rotation_z="3.6651">
-  </xacro:zm_roller_v0>
-  <xacro:zm_roller_v0 prefix="roller_1_8" parent="wheel_1" origin_x="${roller_8_y}" origin_y="${roller_8_x}"
+  </xacro:junbot_roller_v0>
+  <xacro:junbot_roller_v0 prefix="roller_1_8" parent="wheel_1" origin_x="${roller_8_y}" origin_y="${roller_8_x}"
                                                            rotation_x="0.7854" rotation_z="2.967">
-  </xacro:zm_roller_v0>
-  <xacro:zm_roller_v0 prefix="roller_1_9" parent="wheel_1" origin_x="${roller_9_y}" origin_y="${roller_9_x}"
+  </xacro:junbot_roller_v0>
+  <xacro:junbot_roller_v0 prefix="roller_1_9" parent="wheel_1" origin_x="${roller_9_y}" origin_y="${roller_9_x}"
                                                            rotation_x="0.7854" rotation_z="2.2689">
-  </xacro:zm_roller_v0>
-  <!--zm robot LF wheel-->
-  <xacro:zm_wheel_v2 prefix="2" parent="base_link" origin_x="${wheel_before_L}" origin_y="${wheel_left_W}" rotation_x="${wheel_rotationx}">
-  </xacro:zm_wheel_v2>
-  <!--zm robot LF rollor-->
-  <xacro:zm_roller_v0 prefix="roller_2_1" parent="wheel_2" origin_x="${roller_1_x}" origin_y="${roller_1_y}"
+  </xacro:junbot_roller_v0>
+  <!--junbot robot LF wheel-->
+  <xacro:junbot_wheel_v2 prefix="2" parent="base_link" origin_x="${wheel_before_L}" origin_y="${wheel_left_W}" rotation_x="${wheel_rotationx}">
+  </xacro:junbot_wheel_v2>
+  <!--junbot robot LF rollor-->
+  <xacro:junbot_roller_v0 prefix="roller_2_1" parent="wheel_2" origin_x="${roller_1_x}" origin_y="${roller_1_y}"
                                                            rotation_x="-0.7854" rotation_z="0">
-  </xacro:zm_roller_v0>
-  <xacro:zm_roller_v0 prefix="roller_2_2" parent="wheel_2" origin_x="${roller_2_x}" origin_y="${roller_2_y}"
+  </xacro:junbot_roller_v0>
+  <xacro:junbot_roller_v0 prefix="roller_2_2" parent="wheel_2" origin_x="${roller_2_x}" origin_y="${roller_2_y}"
                                                            rotation_x="-0.7854" rotation_z="0.6981">
-  </xacro:zm_roller_v0>
-  <xacro:zm_roller_v0 prefix="roller_2_3" parent="wheel_2" origin_x="${roller_3_x}" origin_y="${roller_3_y}"
+  </xacro:junbot_roller_v0>
+  <xacro:junbot_roller_v0 prefix="roller_2_3" parent="wheel_2" origin_x="${roller_3_x}" origin_y="${roller_3_y}"
                                                            rotation_x="-0.7854" rotation_z="1.3962">
-  </xacro:zm_roller_v0>
-  <xacro:zm_roller_v0 prefix="roller_2_4" parent="wheel_2" origin_x="${roller_4_x}" origin_y="${roller_4_y}"
+  </xacro:junbot_roller_v0>
+  <xacro:junbot_roller_v0 prefix="roller_2_4" parent="wheel_2" origin_x="${roller_4_x}" origin_y="${roller_4_y}"
                                                            rotation_x="-0.7854" rotation_z="2.0943">
-  </xacro:zm_roller_v0>
-  <xacro:zm_roller_v0 prefix="roller_2_5" parent="wheel_2" origin_x="${roller_5_x}" origin_y="${roller_5_y}"
+  </xacro:junbot_roller_v0>
+  <xacro:junbot_roller_v0 prefix="roller_2_5" parent="wheel_2" origin_x="${roller_5_x}" origin_y="${roller_5_y}"
                                                            rotation_x="-0.7854" rotation_z="2.7924">
-  </xacro:zm_roller_v0>
-  <xacro:zm_roller_v0 prefix="roller_2_6" parent="wheel_2" origin_x="${roller_6_x}" origin_y="${roller_6_y}"
+  </xacro:junbot_roller_v0>
+  <xacro:junbot_roller_v0 prefix="roller_2_6" parent="wheel_2" origin_x="${roller_6_x}" origin_y="${roller_6_y}"
                                                            rotation_x="-0.7854" rotation_z="-2.7924">
-  </xacro:zm_roller_v0>
-  <xacro:zm_roller_v0 prefix="roller_2_7" parent="wheel_2" origin_x="${roller_7_x}" origin_y="${roller_7_y}"
+  </xacro:junbot_roller_v0>
+  <xacro:junbot_roller_v0 prefix="roller_2_7" parent="wheel_2" origin_x="${roller_7_x}" origin_y="${roller_7_y}"
                                                            rotation_x="-0.7854" rotation_z="-2.0943">
-  </xacro:zm_roller_v0>
-  <xacro:zm_roller_v0 prefix="roller_2_8" parent="wheel_2" origin_x="${roller_8_x}" origin_y="${roller_8_y}"
+  </xacro:junbot_roller_v0>
+  <xacro:junbot_roller_v0 prefix="roller_2_8" parent="wheel_2" origin_x="${roller_8_x}" origin_y="${roller_8_y}"
                                                            rotation_x="-0.7854" rotation_z="-1.3962">
-  </xacro:zm_roller_v0>
-  <xacro:zm_roller_v0 prefix="roller_2_9" parent="wheel_2" origin_x="${roller_9_x}" origin_y="${roller_9_y}"
+  </xacro:junbot_roller_v0>
+  <xacro:junbot_roller_v0 prefix="roller_2_9" parent="wheel_2" origin_x="${roller_9_x}" origin_y="${roller_9_y}"
                                                            rotation_x="-0.7854" rotation_z="-0.6981">
-  </xacro:zm_roller_v0>
-  <!--zm robot RF wheel-->
-  <xacro:zm_wheel_v3 prefix="3" parent="base_link" origin_x="${wheel_before_L}" origin_y="${wheel_right_W}" rotation_x="${wheel_rotationx}">
-  </xacro:zm_wheel_v3>
-  <!--zm robot RF rollor-->
-  <xacro:zm_roller_v0 prefix="roller_3_1" parent="wheel_3" origin_x="${roller_1_y}" origin_y="${roller_1_x}"
+  </xacro:junbot_roller_v0>
+  <!--junbot robot RF wheel-->
+  <xacro:junbot_wheel_v3 prefix="3" parent="base_link" origin_x="${wheel_before_L}" origin_y="${wheel_right_W}" rotation_x="${wheel_rotationx}">
+  </xacro:junbot_wheel_v3>
+  <!--junbot robot RF rollor-->
+  <xacro:junbot_roller_v0 prefix="roller_3_1" parent="wheel_3" origin_x="${roller_1_y}" origin_y="${roller_1_x}"
                                                            rotation_x="0.7854" rotation_z="1.5708">
-  </xacro:zm_roller_v0>
-  <xacro:zm_roller_v0 prefix="roller_3_2" parent="wheel_3" origin_x="${roller_2_y}" origin_y="${roller_2_x}"
+  </xacro:junbot_roller_v0>
+  <xacro:junbot_roller_v0 prefix="roller_3_2" parent="wheel_3" origin_x="${roller_2_y}" origin_y="${roller_2_x}"
                                                            rotation_x="0.7854" rotation_z="0.8727">
-  </xacro:zm_roller_v0>
-  <xacro:zm_roller_v0 prefix="roller_3_3" parent="wheel_3" origin_x="${roller_3_y}" origin_y="${roller_3_x}"
+  </xacro:junbot_roller_v0>
+  <xacro:junbot_roller_v0 prefix="roller_3_3" parent="wheel_3" origin_x="${roller_3_y}" origin_y="${roller_3_x}"
                                                            rotation_x="0.7854" rotation_z="0.1746">
-  </xacro:zm_roller_v0>
-  <xacro:zm_roller_v0 prefix="roller_3_4" parent="wheel_3" origin_x="${roller_4_y}" origin_y="${roller_4_x}"
+  </xacro:junbot_roller_v0>
+  <xacro:junbot_roller_v0 prefix="roller_3_4" parent="wheel_3" origin_x="${roller_4_y}" origin_y="${roller_4_x}"
                                                            rotation_x="0.7854" rotation_z="-0.5235">
-  </xacro:zm_roller_v0>
-  <xacro:zm_roller_v0 prefix="roller_3_5" parent="wheel_3" origin_x="${roller_5_y}" origin_y="${roller_5_x}"
+  </xacro:junbot_roller_v0>
+  <xacro:junbot_roller_v0 prefix="roller_3_5" parent="wheel_3" origin_x="${roller_5_y}" origin_y="${roller_5_x}"
                                                            rotation_x="0.7854" rotation_z="-1.2216">
-  </xacro:zm_roller_v0>
-  <xacro:zm_roller_v0 prefix="roller_3_6" parent="wheel_3" origin_x="${roller_6_y}" origin_y="${roller_6_x}"
+  </xacro:junbot_roller_v0>
+  <xacro:junbot_roller_v0 prefix="roller_3_6" parent="wheel_3" origin_x="${roller_6_y}" origin_y="${roller_6_x}"
                                                            rotation_x="0.7854" rotation_z="4.3632">
-  </xacro:zm_roller_v0>
-  <xacro:zm_roller_v0 prefix="roller_3_7" parent="wheel_3" origin_x="${roller_7_y}" origin_y="${roller_7_x}"
+  </xacro:junbot_roller_v0>
+  <xacro:junbot_roller_v0 prefix="roller_3_7" parent="wheel_3" origin_x="${roller_7_y}" origin_y="${roller_7_x}"
                                                            rotation_x="0.7854" rotation_z="3.6651">
-  </xacro:zm_roller_v0>
-  <xacro:zm_roller_v0 prefix="roller_3_8" parent="wheel_3" origin_x="${roller_8_y}" origin_y="${roller_8_x}"
+  </xacro:junbot_roller_v0>
+  <xacro:junbot_roller_v0 prefix="roller_3_8" parent="wheel_3" origin_x="${roller_8_y}" origin_y="${roller_8_x}"
                                                            rotation_x="0.7854" rotation_z="2.967">
-  </xacro:zm_roller_v0>
-  <xacro:zm_roller_v0 prefix="roller_3_9" parent="wheel_3" origin_x="${roller_9_y}" origin_y="${roller_9_x}"
+  </xacro:junbot_roller_v0>
+  <xacro:junbot_roller_v0 prefix="roller_3_9" parent="wheel_3" origin_x="${roller_9_y}" origin_y="${roller_9_x}"
                                                            rotation_x="0.7854" rotation_z="2.2689">
-  </xacro:zm_roller_v0>
-  <!--zm robot RR wheel-->
-  <xacro:zm_wheel_v4 prefix="4" parent="base_link" origin_x="${wheel_after_L}" origin_y="${wheel_right_W}" rotation_x="${wheel_rotationx}">
-  </xacro:zm_wheel_v4>
-  <!--zm robot RR rollor-->
-  <xacro:zm_roller_v0 prefix="roller_4_1" parent="wheel_4" origin_x="${roller_1_x}" origin_y="${roller_1_y}"
+  </xacro:junbot_roller_v0>
+  <!--junbot robot RR wheel-->
+  <xacro:junbot_wheel_v4 prefix="4" parent="base_link" origin_x="${wheel_after_L}" origin_y="${wheel_right_W}" rotation_x="${wheel_rotationx}">
+  </xacro:junbot_wheel_v4>
+  <!--junbot robot RR rollor-->
+  <xacro:junbot_roller_v0 prefix="roller_4_1" parent="wheel_4" origin_x="${roller_1_x}" origin_y="${roller_1_y}"
                                                            rotation_x="-0.7854" rotation_z="0">
-  </xacro:zm_roller_v0>
-  <xacro:zm_roller_v0 prefix="roller_4_2" parent="wheel_4" origin_x="${roller_2_x}" origin_y="${roller_2_y}"
+  </xacro:junbot_roller_v0>
+  <xacro:junbot_roller_v0 prefix="roller_4_2" parent="wheel_4" origin_x="${roller_2_x}" origin_y="${roller_2_y}"
                                                            rotation_x="-0.7854" rotation_z="0.6981">
-  </xacro:zm_roller_v0>
-  <xacro:zm_roller_v0 prefix="roller_4_3" parent="wheel_4" origin_x="${roller_3_x}" origin_y="${roller_3_y}"
+  </xacro:junbot_roller_v0>
+  <xacro:junbot_roller_v0 prefix="roller_4_3" parent="wheel_4" origin_x="${roller_3_x}" origin_y="${roller_3_y}"
                                                            rotation_x="-0.7854" rotation_z="1.3962">
-  </xacro:zm_roller_v0>
-  <xacro:zm_roller_v0 prefix="roller_4_4" parent="wheel_4" origin_x="${roller_4_x}" origin_y="${roller_4_y}"
+  </xacro:junbot_roller_v0>
+  <xacro:junbot_roller_v0 prefix="roller_4_4" parent="wheel_4" origin_x="${roller_4_x}" origin_y="${roller_4_y}"
                                                            rotation_x="-0.7854" rotation_z="2.0943">
-  </xacro:zm_roller_v0>
-  <xacro:zm_roller_v0 prefix="roller_4_5" parent="wheel_4" origin_x="${roller_5_x}" origin_y="${roller_5_y}"
+  </xacro:junbot_roller_v0>
+  <xacro:junbot_roller_v0 prefix="roller_4_5" parent="wheel_4" origin_x="${roller_5_x}" origin_y="${roller_5_y}"
                                                            rotation_x="-0.7854" rotation_z="2.7924">
-  </xacro:zm_roller_v0>
-  <xacro:zm_roller_v0 prefix="roller_4_6" parent="wheel_4" origin_x="${roller_6_x}" origin_y="${roller_6_y}"
+  </xacro:junbot_roller_v0>
+  <xacro:junbot_roller_v0 prefix="roller_4_6" parent="wheel_4" origin_x="${roller_6_x}" origin_y="${roller_6_y}"
                                                            rotation_x="-0.7854" rotation_z="-2.7924">
-  </xacro:zm_roller_v0>
-  <xacro:zm_roller_v0 prefix="roller_4_7" parent="wheel_4" origin_x="${roller_7_x}" origin_y="${roller_7_y}"
+  </xacro:junbot_roller_v0>
+  <xacro:junbot_roller_v0 prefix="roller_4_7" parent="wheel_4" origin_x="${roller_7_x}" origin_y="${roller_7_y}"
                                                            rotation_x="-0.7854" rotation_z="-2.0943">
-  </xacro:zm_roller_v0>
-  <xacro:zm_roller_v0 prefix="roller_4_8" parent="wheel_4" origin_x="${roller_8_x}" origin_y="${roller_8_y}"
+  </xacro:junbot_roller_v0>
+  <xacro:junbot_roller_v0 prefix="roller_4_8" parent="wheel_4" origin_x="${roller_8_x}" origin_y="${roller_8_y}"
                                                            rotation_x="-0.7854" rotation_z="-1.3962">
-  </xacro:zm_roller_v0>
-  <xacro:zm_roller_v0 prefix="roller_4_9" parent="wheel_4" origin_x="${roller_9_x}" origin_y="${roller_9_y}"
+  </xacro:junbot_roller_v0>
+  <xacro:junbot_roller_v0 prefix="roller_4_9" parent="wheel_4" origin_x="${roller_9_x}" origin_y="${roller_9_y}"
                                                            rotation_x="-0.7854" rotation_z="-0.6981">
-  </xacro:zm_roller_v0>
+  </xacro:junbot_roller_v0>
   <!-- Wheel -->
   <xacro:wheel_gazebo_v0 prefix="1"/>
@@ -401,15 +401,15 @@
   <xacro:roller_trans_v0 prefix="roller_4_9"/>
   <!-- ultrasound
-  <xacro:zm_ultrasound prefix="1" parent="base_link" origin_x="${ul_left_front_x}" origin_y="${ul_left_front_y}"
+  <xacro:junbot_ultrasound prefix="1" parent="base_link" origin_x="${ul_left_front_x}" origin_y="${ul_left_front_y}"
                                                      origin_z="${ul_hight}" rotation_z="${ul_front_rotation}">
-  </xacro:zm_ultrasound>
-  <xacro:zm_ultrasound prefix="2" parent="base_link" origin_x="${ul_right_front_x}" origin_y="${ul_right_front_y}"
+  </xacro:junbot_ultrasound>
+  <xacro:junbot_ultrasound prefix="2" parent="base_link" origin_x="${ul_right_front_x}" origin_y="${ul_right_front_y}"
                                                      origin_z="${ul_hight}" rotation_z="${ul_front_rotation}">
-  </xacro:zm_ultrasound>
-  <xacro:zm_ultrasound prefix="3" parent="base_link" origin_x="${ul_left_rear_x}" origin_y="${ul_left_rear_y}"
+  </xacro:junbot_ultrasound>
+  <xacro:junbot_ultrasound prefix="3" parent="base_link" origin_x="${ul_left_rear_x}" origin_y="${ul_left_rear_y}"
                                                      origin_z="${ul_hight}" rotation_z="${ul_rear_rotation}">
-  </xacro:zm_ultrasound>
-  <xacro:zm_ultrasound prefix="4" parent="base_link" origin_x="${ul_right_rear_x}" origin_y="${ul_right_rear_y}"
+  </xacro:junbot_ultrasound>
+  <xacro:junbot_ultrasound prefix="4" parent="base_link" origin_x="${ul_right_rear_x}" origin_y="${ul_right_rear_y}"
                                                      origin_z="${ul_hight}" rotation_z="${ul_rear_rotation}">
-  </xacro:zm_ultrasound> -->
+  </xacro:junbot_ultrasound> -->
 </robot>

File: junbot/junbot_description/urdf/junbot_roller.urdf.xacro (robot description, xacro)
@@ -3,5 +3,5 @@
   <xacro:include filename="$(find junbot_description)/urdf/junbot_roller.transmission.xacro"/>
   <xacro:include filename="$(find junbot_description)/urdf/junbot_roller.gazebo"/>
-  <xacro:macro name="zm_roller_v0" params="prefix parent origin_x origin_y rotation_x rotation_z">
+  <xacro:macro name="junbot_roller_v0" params="prefix parent origin_x origin_y rotation_x rotation_z">
 	<joint name="${prefix}_joint" type="continuous">
 	  <parent link="${parent}"/>

File: junbot/junbot_description/urdf/junbot_ultrasound.urdf.xacro (robot description, xacro)
@@ -2,5 +2,5 @@
 <robot xmlns:xacro="http://ros.org/wiki/xacro">
   <xacro:include filename="$(find junbot_description)/urdf/junbot_ultrasound.gazebo"/>
-  <xacro:macro name="zm_ultrasound" params="prefix parent origin_x origin_y origin_z rotation_z">
+  <xacro:macro name="junbot_ultrasound" params="prefix parent origin_x origin_y origin_z rotation_z">
 	<joint name="ultrasound_joint_${prefix}" type="fixed">
 	  <parent link="${parent}"/>

File: junbot/junbot_description/urdf/junbot_wheel_LF.urdf.xacro (robot description, xacro)
@@ -2,5 +2,5 @@
 <robot xmlns:xacro="http://ros.org/wiki/xacro">
   <xacro:include filename="$(find junbot_description)/urdf/junbot_wheel.gazebo"/>
-  <xacro:macro name="zm_wheel_v2" params="prefix parent origin_x origin_y rotation_x">
+  <xacro:macro name="junbot_wheel_v2" params="prefix parent origin_x origin_y rotation_x">
 	<joint name="wheel_joint_${prefix}" type="continuous">
 	  <parent link="${parent}"/>

File: junbot/junbot_description/urdf/junbot_wheel_LR.urdf.xacro (robot description, xacro)
@@ -2,5 +2,5 @@
 <robot xmlns:xacro="http://ros.org/wiki/xacro">
   <xacro:include filename="$(find junbot_description)/urdf/junbot_wheel.gazebo"/>
-  <xacro:macro name="zm_wheel_v1" params="prefix parent origin_x origin_y rotation_x">
+  <xacro:macro name="junbot_wheel_v1" params="prefix parent origin_x origin_y rotation_x">
 	<joint name="wheel_joint_${prefix}" type="continuous">
 	  <parent link="${parent}"/>

File: junbot/junbot_description/urdf/junbot_wheel_RF.urdf.xacro (robot description, xacro)
@@ -2,5 +2,5 @@
 <robot xmlns:xacro="http://ros.org/wiki/xacro">
   <xacro:include filename="$(find junbot_description)/urdf/junbot_wheel.gazebo"/>
-  <xacro:macro name="zm_wheel_v3" params="prefix parent origin_x origin_y rotation_x">
+  <xacro:macro name="junbot_wheel_v3" params="prefix parent origin_x origin_y rotation_x">
 	<joint name="wheel_joint_${prefix}" type="continuous">
 	  <parent link="${parent}"/>

File: junbot/junbot_description/urdf/junbot_wheel_RR.urdf.xacro (robot description, xacro)
@@ -2,5 +2,5 @@
 <robot xmlns:xacro="http://ros.org/wiki/xacro">
   <xacro:include filename="$(find junbot_description)/urdf/junbot_wheel.gazebo"/>
-  <xacro:macro name="zm_wheel_v4" params="prefix parent origin_x origin_y rotation_x">
+  <xacro:macro name="junbot_wheel_v4" params="prefix parent origin_x origin_y rotation_x">
 	<joint name="wheel_joint_${prefix}" type="continuous">
 	  <parent link="${parent}"/>

Commit message: [Added] add rplidar a2

File: junbot/junbot_description/urdf/junbot_mecanum.urdf.xacro (robot description, xacro)
@@ -140,15 +140,15 @@
   </link> -->
   <!-- kinect V2 -->
-  <joint name="kinect_v2_joint " type="fixed">
+  <joint name="t265_joint " type="fixed">
     <parent link="base_link"/>
-    <child link="kinect_v2"/>
+    <child link="t265"/>
     <origin xyz="0.33 0 0.122015" rpy="0 0 0"/>
     <axis xyz="0 0 1"/>
   </joint>
-  <link name="kinect_v2">
+  <link name="t265">
     <collision>
       <origin xyz="0 0 0" rpy="0 0 0"/>
       <geometry>
-	      <mesh filename="package://junbot_description/meshes/kinect_v2.stl" scale="0.01 0.01 0.01"/>
+	      <mesh filename="package://junbot_description/meshes/t265.stl" scale="0.01 0.01 0.01"/>
       </geometry>
     </collision>
@@ -156,5 +156,5 @@
       <origin xyz="0 0 0" rpy="0 0 0"/>
       <geometry>
-	      <mesh filename="package://junbot_description/meshes/kinect_v2.stl" scale="0.01 0.01 0.01"/>
+	      <mesh filename="package://junbot_description/meshes/t265.stl" scale="0.01 0.01 0.01"/>
       </geometry>
       <material name="black"/>

Commit message: [fixed] fix frame odom to  t265 odom for navigation

File: junbot/junbot_description/urdf/junbot_mecanum.urdf.xacro (robot description, xacro)
@@ -84,10 +84,10 @@
   </link>
   <!-- sick LiDAR 0 -->
-  <joint name="sick_lidar0_joint" type="fixed">
+  <joint name="scan_joint" type="fixed">
     <parent link="base_link"/>
-    <child link="sick_lidar0"/>
+    <child link="laser"/>
     <origin xyz="0.2 0 0.195722" rpy="0 0 0"/>
   </joint>
-  <link name="sick_lidar0">
+  <link name="laser">
     <collision>
       <origin xyz="0 0 0" rpy="0 0 0"/>
@@ -141,10 +141,10 @@
   <!-- kinect V2 -->
   <joint name="t265_joint " type="fixed">
-    <parent link="base_link"/>
-    <child link="t265"/>
+    <parent link="base_footprint"/>
+    <child link="t265_link"/>
     <origin xyz="0.33 0 0.122015" rpy="0 0 0"/>
     <axis xyz="0 0 1"/>
   </joint>
-  <link name="t265">
+  <link name="t265_link">
     <collision>
       <origin xyz="0 0 0" rpy="0 0 0"/>
@@ -169,5 +169,5 @@
   </link>
   <!-- IMU -->
-  <joint name="IMU_joint " type="fixed">
+  <!-- <joint name="IMU_joint " type="fixed">
     <parent link="base_link"/>
     <child link="IMU_sensor"/>
@@ -196,5 +196,5 @@
 	            izz="0.00005"/>
     </inertial>
-  </link>
+  </link> -->
   <!--junbot robot LR wheel-->
   <xacro:junbot_wheel_v1 prefix="1" parent="base_link" origin_x="${wheel_after_L}" origin_y="${wheel_left_W}" rotation_x="${wheel_rotationx}">
